Commit message: update 2d xacro file

File: simulation/urdf/mikkelsen2d_description/urdf/mikkelsen2d.xacro (robot description, xacro)
@@ -4,1024 +4,4 @@
 <xacro:include filename="$(find mikkelsen2d_description)/urdf/mikkelsen2d.trans" />
 <xacro:include filename="$(find mikkelsen2d_description)/urdf/mikkelsen2d.gazebo" />
-<link name="base_link">
-  <inertial>
-    <origin xyz="-0.037679135816683924 0.012666740518570965 -0.058008954907279954" rpy="0 0 0"/>
-    <mass value="0.42566063723793834"/>
-    <inertia ixx="0.000885" iyy="0.000452" izz="0.000847" ixy="3.1e-05" iyz="1e-06" ixz="-7e-06"/>
-  </inertial>
-  <visual>
-    <origin xyz="0 0 0" rpy="0 0 0"/>
-    <geometry>
-      <mesh filename="package://mikkelsen2d_description/meshes/base_link.stl" scale="0.001 0.001 0.001"/>
-    </geometry>
-    <material name="pa_11_nylon_hp_1130_eos_p_396_3d_"/>
-  </visual>
-  <collision>
-    <origin xyz="0 0 0" rpy="0 0 0"/>
-    <geometry>
-      <mesh filename="package://mikkelsen2d_description/meshes/base_link.stl" scale="0.001 0.001 0.001"/>
-    </geometry>
-  </collision>
-</link>
-<link name="R_hip_roll_xl_2">
-  <inertial>
-    <origin xyz="-0.004986268827101341 -0.014720443125513842 -0.015885149307033275" rpy="0 0 0"/>
-    <mass value="0.040973661549071165"/>
-    <inertia ixx="1e-05" iyy="1.1e-05" izz="6e-06" ixy="-0.0" iyz="-0.0" ixz="0.0"/>
-  </inertial>
-  <visual>
-    <origin xyz="0.023805 0.046388 0.034586" rpy="0 0 0"/>
-    <geometry>
-      <mesh filename="package://mikkelsen2d_description/meshes/R_hip_roll_xl_2.stl" scale="0.001 0.001 0.001"/>
-    </geometry>
-    <material name=""/>
-  </visual>
-  <collision>
-    <origin xyz="0.023805 0.046388 0.034586" rpy="0 0 0"/>
-    <geometry>
-      <mesh filename="package://mikkelsen2d_description/meshes/R_hip_roll_xl_2.stl" scale="0.001 0.001 0.001"/>
-    </geometry>
-  </collision>
-</link>
-<link name="R_hip_roll_2">
-  <inertial>
-    <origin xyz="0.016632013644877517 0.0012074494935598173 0.0006988114411143054" rpy="0 0 0"/>
-    <mass value="0.001436423594975712"/>
-    <inertia ixx="0.0" iyy="0.0" izz="0.0" ixy="-0.0" iyz="-0.0" ixz="-0.0"/>
-  </inertial>
-  <visual>
-    <origin xyz="0.044871 0.062309 0.0632" rpy="0 0 0"/>
-    <geometry>
-      <mesh filename="package://mikkelsen2d_description/meshes/R_hip_roll_2.stl" scale="0.001 0.001 0.001"/>
-    </geometry>
-    <material name=""/>
-  </visual>
-  <collision>
-    <origin xyz="0.044871 0.062309 0.0632" rpy="0 0 0"/>
-    <geometry>
-      <mesh filename="package://mikkelsen2d_description/meshes/R_hip_roll_2.stl" scale="0.001 0.001 0.001"/>
-    </geometry>
-  </collision>
-</link>
-<link name="hip_roll_bracket_1">
-  <inertial>
-    <origin xyz="-0.005977579788513737 -0.0004317805669656269 -0.00017873596901929467" rpy="0 0 0"/>
-    <mass value="0.005303897131480488"/>
-    <inertia ixx="1e-06" iyy="1e-06" izz="1e-06" ixy="0.0" iyz="0.0" ixz="0.0"/>
-  </inertial>
-  <visual>
-    <origin xyz="0.046865 0.062453 0.063259" rpy="0 0 0"/>
-    <geometry>
-      <mesh filename="package://mikkelsen2d_description/meshes/hip_roll_bracket_1.stl" scale="0.001 0.001 0.001"/>
-    </geometry>
-    <material name="pa_11_nylon_hp_1130_eos_p_396_3d_"/>
-  </visual>
-  <collision>
-    <origin xyz="0.046865 0.062453 0.063259" rpy="0 0 0"/>
-    <geometry>
-      <mesh filename="package://mikkelsen2d_description/meshes/hip_roll_bracket_1.stl" scale="0.001 0.001 0.001"/>
-    </geometry>
-  </collision>
-</link>
-<link name="R_hip_yaw_xl_2">
-  <inertial>
-    <origin xyz="-0.006998679111861819 -0.014828044606016055 -0.006688075872869702" rpy="0 0 0"/>
-    <mass value="0.040973661549071165"/>
-    <inertia ixx="6e-06" iyy="1.1e-05" izz="1e-05" ixy="-0.0" iyz="-0.0" ixz="-0.0"/>
-  </inertial>
-  <visual>
-    <origin xyz="0.065267 0.049471 0.057833" rpy="0 0 0"/>
-    <geometry>
-      <mesh filename="package://mikkelsen2d_description/meshes/R_hip_yaw_xl_2.stl" scale="0.001 0.001 0.001"/>
-    </geometry>
-    <material name=""/>
-  </visual>
-  <collision>
-    <origin xyz="0.065267 0.049471 0.057833" rpy="0 0 0"/>
-    <geometry>
-      <mesh filename="package://mikkelsen2d_description/meshes/R_hip_yaw_xl_2.stl" scale="0.001 0.001 0.001"/>
-    </geometry>
-  </collision>
-</link>
-<link name="R_hip_yaw_2">
-  <inertial>
-    <origin xyz="-0.0007020290665685561 2.278650526520154e-05 0.01667620487029814" rpy="0 0 0"/>
-    <mass value="0.001436423594975712"/>
-    <inertia ixx="0.0" iyy="0.0" izz="0.0" ixy="0.0" iyz="-0.0" ixz="0.0"/>
-  </inertial>
-  <visual>
-    <origin xyz="0.059566 0.063439 0.080646" rpy="0 0 0"/>
-    <geometry>
-      <mesh filename="package://mikkelsen2d_description/meshes/R_hip_yaw_2.stl" scale="0.001 0.001 0.001"/>
-    </geometry>
-    <material name=""/>
-  </visual>
-  <collision>
-    <origin xyz="0.059566 0.063439 0.080646" rpy="0 0 0"/>
-    <geometry>
-      <mesh filename="package://mikkelsen2d_description/meshes/R_hip_yaw_2.stl" scale="0.001 0.001 0.001"/>
-    </geometry>
-  </collision>
-</link>
-<link name="hip_yaw_bracket_1">
-  <inertial>
-    <origin xyz="-0.001846672263714419 -0.00015526908116847427 -0.005510024391643234" rpy="0 0 0"/>
-    <mass value="0.0070036931272659"/>
-    <inertia ixx="1e-06" iyy="1e-06" izz="2e-06" ixy="-0.0" iyz="-0.0" ixz="-0.0"/>
-  </inertial>
-  <visual>
-    <origin xyz="0.059506 0.063443 0.082645" rpy="0 0 0"/>
-    <geometry>
-      <mesh filename="package://mikkelsen2d_description/meshes/hip_yaw_bracket_1.stl" scale="0.001 0.001 0.001"/>
-    </geometry>
-    <material name="pa_11_nylon_hp_1130_eos_p_396_3d_"/>
-  </visual>
-  <collision>
-    <origin xyz="0.059506 0.063443 0.082645" rpy="0 0 0"/>
-    <geometry>
-      <mesh filename="package://mikkelsen2d_description/meshes/hip_yaw_bracket_1.stl" scale="0.001 0.001 0.001"/>
-    </geometry>
-  </collision>
-</link>
-<link name="R_hip_pitch_xl_2">
-  <inertial>
-    <origin xyz="-0.0034402792651398242 -0.005843576841470306 -0.02087676372452038" rpy="0 0 0"/>
-    <mass value="0.040973661549071165"/>
-    <inertia ixx="1e-05" iyy="1e-05" izz="8e-06" ixy="-0.0" iyz="0.0" ixz="2e-06"/>
-  </inertial>
-  <visual>
-    <origin xyz="0.040306 0.056066 0.088365" rpy="0 0 0"/>
-    <geometry>
-      <mesh filename="package://mikkelsen2d_description/meshes/R_hip_pitch_xl_2.stl" scale="0.001 0.001 0.001"/>
-    </geometry>
-    <material name=""/>
-  </visual>
-  <collision>
-    <origin xyz="0.040306 0.056066 0.088365" rpy="0 0 0"/>
-    <geometry>
-      <mesh filename="package://mikkelsen2d_description/meshes/R_hip_pitch_xl_2.stl" scale="0.001 0.001 0.001"/>
-    </geometry>
-  </collision>
-</link>
-<link name="R_hip_pitch_2">
-  <inertial>
-    <origin xyz="0.0010986594270186306 -0.016652648300792397 0.0002431266431453527" rpy="0 0 0"/>
-    <mass value="0.001436423594975712"/>
-    <inertia ixx="0.0" iyy="0.0" izz="0.0" ixy="0.0" iyz="0.0" ixz="-0.0"/>
-  </inertial>
-  <visual>
-    <origin xyz="0.038503 0.045035 0.11972" rpy="0 0 0"/>
-    <geometry>
-      <mesh filename="package://mikkelsen2d_description/meshes/R_hip_pitch_2.stl" scale="0.001 0.001 0.001"/>
-    </geometry>
-    <material name=""/>
-  </visual>
-  <collision>
-    <origin xyz="0.038503 0.045035 0.11972" rpy="0 0 0"/>
-    <geometry>
-      <mesh filename="package://mikkelsen2d_description/meshes/R_hip_pitch_2.stl" scale="0.001 0.001 0.001"/>
-    </geometry>
-  </collision>
-</link>
-<link name="hip_pitch_bracket_1">
-  <inertial>
-    <origin xyz="0.0075391568599490685 -0.018546209284858436 -0.009937387556057525" rpy="0 0 0"/>
-    <mass value="0.005694190208798132"/>
-    <inertia ixx="2e-06" iyy="1e-06" izz="2e-06" ixy="0.0" iyz="0.0" ixz="0.0"/>
-  </inertial>
-  <visual>
-    <origin xyz="0.038647 0.04304 0.119728" rpy="0 0 0"/>
-    <geometry>
-      <mesh filename="package://mikkelsen2d_description/meshes/hip_pitch_bracket_1.stl" scale="0.001 0.001 0.001"/>
-    </geometry>
-    <material name="pa_11_nylon_hp_1130_eos_p_396_3d_"/>
-  </visual>
-  <collision>
-    <origin xyz="0.038647 0.04304 0.119728" rpy="0 0 0"/>
-    <geometry>
-      <mesh filename="package://mikkelsen2d_description/meshes/hip_pitch_bracket_1.stl" scale="0.001 0.001 0.001"/>
-    </geometry>
-  </collision>
-</link>
-<link name="R_knee_xl_2">
-  <inertial>
-    <origin xyz="0.005665122216174493 -0.00519891645315862 -0.02376072216402675" rpy="0 0 0"/>
-    <mass value="0.040973661549071165"/>
-    <inertia ixx="1e-05" iyy="1e-05" izz="8e-06" ixy="-0.0" iyz="0.0" ixz="2e-06"/>
-  </inertial>
-  <visual>
-    <origin xyz="0.020568 0.054821 0.132273" rpy="0 0 0"/>
-    <geometry>
-      <mesh filename="package://mikkelsen2d_description/meshes/R_knee_xl_2.stl" scale="0.001 0.001 0.001"/>
-    </geometry>
-    <material name=""/>
-  </visual>
-  <collision>
-    <origin xyz="0.020568 0.054821 0.132273" rpy="0 0 0"/>
-    <geometry>
-      <mesh filename="package://mikkelsen2d_description/meshes/R_knee_xl_2.stl" scale="0.001 0.001 0.001"/>
-    </geometry>
-  </collision>
-</link>
-<link name="R_knee_2">
-  <inertial>
-    <origin xyz="0.0010990609083328055 -0.016652987912480627 0.0002431682036394267" rpy="0 0 0"/>
-    <mass value="0.001436423594975712"/>
-    <inertia ixx="0.0" iyy="0.0" izz="0.0" ixy="0.0" iyz="0.0" ixz="-0.0"/>
-  </inertial>
-  <visual>
-    <origin xyz="0.00966 0.043145 0.166512" rpy="0 0 0"/>
-    <geometry>
-      <mesh filename="package://mikkelsen2d_description/meshes/R_knee_2.stl" scale="0.001 0.001 0.001"/>
-    </geometry>
-    <material name=""/>
-  </visual>
-  <collision>
-    <origin xyz="0.00966 0.043145 0.166512" rpy="0 0 0"/>
-    <geometry>
-      <mesh filename="package://mikkelsen2d_description/meshes/R_knee_2.stl" scale="0.001 0.001 0.001"/>
-    </geometry>
-  </collision>
-</link>
-<link name="knee_r_brecket_1">
-  <inertial>
-    <origin xyz="0.009880315866068638 -0.007544733859495598 -0.0235916808233316" rpy="0 0 0"/>
-    <mass value="0.00786109169007575"/>
-    <inertia ixx="1e-06" iyy="1e-06" izz="1e-06" ixy="0.0" iyz="-0.0" ixz="0.0"/>
-  </inertial>
-  <visual>
-    <origin xyz="0.009804 0.04115 0.16652" rpy="0 0 0"/>
-    <geometry>
-      <mesh filename="package://mikkelsen2d_description/meshes/knee_r_brecket_1.stl" scale="0.001 0.001 0.001"/>
-    </geometry>
-    <material name="pa_11_nylon_hp_1130_eos_p_396_3d_"/>
-  </visual>
-  <collision>
-    <origin xyz="0.009804 0.04115 0.16652" rpy="0 0 0"/>
-    <geometry>
-      <mesh filename="package://mikkelsen2d_description/meshes/knee_r_brecket_1.stl" scale="0.001 0.001 0.001"/>
-    </geometry>
-  </collision>
-</link>
-<link name="leg_upper_1">
-  <inertial>
-    <origin xyz="-0.0236265091226358 -0.0018811073277059803 -0.044025157686495536" rpy="0 0 0"/>
-    <mass value="0.012719491840295135"/>
-    <inertia ixx="8e-06" iyy="1.1e-05" izz="3e-06" ixy="-0.0" iyz="-0.0" ixz="-4e-06"/>
-  </inertial>
-  <visual>
-    <origin xyz="-0.00337 0.052837 0.192104" rpy="0 0 0"/>
-    <geometry>
-      <mesh filename="package://mikkelsen2d_description/meshes/leg_upper_1.stl" scale="0.001 0.001 0.001"/>
-    </geometry>
-    <material name="pa_11_nylon_hp_1130_eos_p_396_3d_"/>
-  </visual>
-  <collision>
-    <origin xyz="-0.00337 0.052837 0.192104" rpy="0 0 0"/>
-    <geometry>
-      <mesh filename="package://mikkelsen2d_description/meshes/leg_upper_1.stl" scale="0.001 0.001 0.001"/>
-    </geometry>
-  </collision>
-</link>
-<link name="lower_knee_link_2">
-  <inertial>
-    <origin xyz="0.0053390673542219255 0.00037288933482495373 -0.003360765157294665" rpy="0 0 0"/>
-    <mass value="0.010036812614450108"/>
-    <inertia ixx="1e-06" iyy="2e-06" izz="1e-06" ixy="-0.0" iyz="0.0" ixz="0.0"/>
-  </inertial>
-  <visual>
-    <origin xyz="0.043883 0.056599 0.280155" rpy="0 0 0"/>
-    <geometry>
-      <mesh filename="package://mikkelsen2d_description/meshes/lower_knee_link_2.stl" scale="0.001 0.001 0.001"/>
-    </geometry>
-    <material name="pa_11_nylon_hp_1130_eos_p_396_3d_"/>
-  </visual>
-  <collision>
-    <origin xyz="0.043883 0.056599 0.280155" rpy="0 0 0"/>
-    <geometry>
-      <mesh filename="package://mikkelsen2d_description/meshes/lower_knee_link_2.stl" scale="0.001 0.001 0.001"/>
-    </geometry>
-  </collision>
-</link>
-<link name="R_ankle_xl_2">
-  <inertial>
-    <origin xyz="0.0023787863497140467 -0.14124852441426808 -0.013927891020301064" rpy="0 0 0"/>
-    <mass value="0.040973661549071165"/>
-    <inertia ixx="1e-05" iyy="1e-05" izz="8e-06" ixy="-0.0" iyz="0.0" ixz="2e-06"/>
-  </inertial>
-  <visual>
-    <origin xyz="0.026284 -0.086403 0.292492" rpy="0 0 0"/>
-    <geometry>
-      <mesh filename="package://mikkelsen2d_description/meshes/R_ankle_xl_2.stl" scale="0.001 0.001 0.001"/>
-    </geometry>
-    <material name=""/>
-  </visual>
-  <collision>
-    <origin xyz="0.026284 -0.086403 0.292492" rpy="0 0 0"/>
-    <geometry>
-      <mesh filename="package://mikkelsen2d_description/meshes/R_ankle_xl_2.stl" scale="0.001 0.001 0.001"/>
-    </geometry>
-  </collision>
-</link>
-<link name="R_ankle_2">
-  <inertial>
-    <origin xyz="0.0013006383168733017 -0.016639995225795144 -0.00010822058159531966" rpy="0 0 0"/>
-    <mass value="0.001436423594975712"/>
-    <inertia ixx="0.0" iyy="0.0" izz="0.0" ixy="0.0" iyz="-0.0" ixz="0.0"/>
-  </inertial>
-  <visual>
-    <origin xyz="0.03152 0.038813 0.296075" rpy="0 0 0"/>
-    <geometry>
-      <mesh filename="package://mikkelsen2d_description/meshes/R_ankle_2.stl" scale="0.001 0.001 0.001"/>
-    </geometry>
-    <material name=""/>
-  </visual>
-  <collision>
-    <origin xyz="0.03152 0.038813 0.296075" rpy="0 0 0"/>
-    <geometry>
-      <mesh filename="package://mikkelsen2d_description/meshes/R_ankle_2.stl" scale="0.001 0.001 0.001"/>
-    </geometry>
-  </collision>
-</link>
-<link name="ankle_link_1_2">
-  <inertial>
-    <origin xyz="-0.01962001103280569 -0.009168861831198263 -0.012464641305166724" rpy="0 0 0"/>
-    <mass value="0.006084906833817184"/>
-    <inertia ixx="1e-06" iyy="1e-06" izz="1e-06" ixy="-0.0" iyz="-0.0" ixz="-0.0"/>
-  </inertial>
-  <visual>
-    <origin xyz="0.031664 0.036818 0.296083" rpy="0 0 0"/>
-    <geometry>
-      <mesh filename="package://mikkelsen2d_description/meshes/ankle_link_1_2.stl" scale="0.001 0.001 0.001"/>
-    </geometry>
-    <material name="pa_11_nylon_hp_1130_eos_p_396_3d_"/>
-  </visual>
-  <collision>
-    <origin xyz="0.031664 0.036818 0.296083" rpy="0 0 0"/>
-    <geometry>
-      <mesh filename="package://mikkelsen2d_description/meshes/ankle_link_1_2.stl" scale="0.001 0.001 0.001"/>
-    </geometry>
-  </collision>
-</link>
-<link name="ankle_link_2_2">
-  <inertial>
-    <origin xyz="-0.018515664582423236 0.0026780261680551254 -0.011305066027976263" rpy="0 0 0"/>
-    <mass value="0.004445165114646534"/>
-    <inertia ixx="0.0" iyy="1e-06" izz="1e-06" ixy="0.0" iyz="0.0" ixz="-0.0"/>
-  </inertial>
-  <visual>
-    <origin xyz="0.028932 0.07472 0.29593" rpy="0 0 0"/>
-    <geometry>
-      <mesh filename="package://mikkelsen2d_description/meshes/ankle_link_2_2.stl" scale="0.001 0.001 0.001"/>
-    </geometry>
-    <material name="pa_11_nylon_hp_1130_eos_p_396_3d_"/>
-  </visual>
-  <collision>
-    <origin xyz="0.028932 0.07472 0.29593" rpy="0 0 0"/>
-    <geometry>
-      <mesh filename="package://mikkelsen2d_description/meshes/ankle_link_2_2.stl" scale="0.001 0.001 0.001"/>
-    </geometry>
-  </collision>
-</link>
-<link name="R_bionic_biped_robot_ankle_bar_1">
-  <inertial>
-    <origin xyz="0.0372744305641953 -0.13529755106127062 -0.03135385985193945" rpy="0 0 0"/>
-    <mass value="0.003337002701996774"/>
-    <inertia ixx="2e-06" iyy="3e-06" izz="1e-06" ixy="-0.0" iyz="0.0" ixz="1e-06"/>
-  </inertial>
-  <visual>
-    <origin xyz="0.065636 -0.079475 0.312328" rpy="0 0 0"/>
-    <geometry>
-      <mesh filename="package://mikkelsen2d_description/meshes/R_bionic_biped_robot_ankle_bar_1.stl" scale="0.001 0.001 0.001"/>
-    </geometry>
-    <material name="pa_11_nylon_hp_1130_eos_p_396_3d_"/>
-  </visual>
-  <collision>
-    <origin xyz="0.065636 -0.079475 0.312328" rpy="0 0 0"/>
-    <geometry>
-      <mesh filename="package://mikkelsen2d_description/meshes/R_bionic_biped_robot_ankle_bar_1.stl" scale="0.001 0.001 0.001"/>
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
Commit message: update dql

File: simulation/urdf/mikkelsen2d_description/urdf/mikkelsen2d.xacro (robot description, xacro)
@@ -13,5 +13,5 @@
 <link name="z_prismatic">
   <inertial>
-    <mass value="40"/>
+    <mass value="35"/>
     <inertia ixx="0.2125" ixy="-0.005" ixz="0.0225" iyy="0.205" iyz="0.045" izz="0.0125"/>
     <origin rpy="0 0 0" xyz="0 0 0"/>

Commit message: update dql

File: simulation/urdf/mikkelsen2d_description/urdf/mikkelsen2d.xacro (robot description, xacro)
@@ -13,5 +13,5 @@
 <link name="z_prismatic">
   <inertial>
-    <mass value="35"/>
+    <mass value="50"/>
     <inertia ixx="0.2125" ixy="-0.005" ixz="0.0225" iyy="0.205" iyz="0.045" izz="0.0125"/>
     <origin rpy="0 0 0" xyz="0 0 0"/>

Commit message: update closed link

File: simulation/urdf/mikkelsen2d_description/urdf/mikkelsen2d.xacro (robot description, xacro)
@@ -13,5 +13,5 @@
 <link name="z_prismatic">
   <inertial>
-    <mass value="50"/>
+    <mass value="100"/>
     <inertia ixx="0.2125" ixy="-0.005" ixz="0.0225" iyy="0.205" iyz="0.045" izz="0.0125"/>
     <origin rpy="0 0 0" xyz="0 0 0"/>
@@ -1065,4 +1065,18 @@
   </collision>
 </link>
+<joint name="��] 249" type="revolute">
+  <origin xyz="0.010519 -0.134088 0.001069" rpy="0 0 0"/>
+  <parent link="shaft_1"/>
+  <child link="foot_1"/>
+  <axis xyz="-0.071895 0.997404 -0.004038"/>
+  <limit lower="-0.5236" upper="0.5236" effort="100" velocity="1.0"/>
+</joint>
+<joint name="��] 292" type="revolute">
+  <origin xyz="0.010662 -0.136083 0.001077" rpy="0 0 0"/>
+  <parent link="shaft_4"/>
+  <child link="foot_2"/>
+  <axis xyz="-0.071895 0.997404 -0.004038"/>
+  <limit lower="-0.5236" upper="0.5236" effort="100" velocity="1.0"/>
+</joint>
 <joint name="���� 226" type="fixed">
   <origin xyz="-0.023805 -0.046388 -0.034586" rpy="0 0 0"/>
@@ -1185,10 +1199,4 @@
   <child link="shaft_1"/>
 </joint>
-<joint name="��] 249" type="continuous">
-  <origin xyz="0.010519 -0.134088 0.001069" rpy="0 0 0"/>
-  <parent link="shaft_1"/>
-  <child link="foot_1"/>
-  <axis xyz="-0.071895 0.997404 -0.004038"/>
-</joint>
 <joint name="���� 270" type="fixed">
   <origin xyz="-0.032432 0.073301 -0.03507" rpy="0 0 0"/>
@@ -1305,10 +1313,4 @@
   <child link="shaft_4"/>
 </joint>
-<joint name="��] 292" type="continuous">
-  <origin xyz="0.010662 -0.136083 0.001077" rpy="0 0 0"/>
-  <parent link="shaft_4"/>
-  <child link="foot_2"/>
-  <axis xyz="-0.071895 0.997404 -0.004038"/>
-</joint>
 <joint name="��] 294" type="continuous">
   <origin xyz="0.062297 0.000176 -0.074829" rpy="0 0 0"/>

Commit message: update closed link and datasaver

File: simulation/urdf/mikkelsen2d_description/urdf/mikkelsen2d.xacro (robot description, xacro)
@@ -1065,4 +1065,46 @@
   </collision>
 </link>
+<joint name="��] 241" type="revolute">
+  <origin xyz="-0.005236 -0.125216 -0.003583" rpy="0 0 0"/>
+  <parent link="R_ankle_xl_2"/>
+  <child link="R_ankle_2"/>
+  <axis xyz="0.071895 -0.997404 0.004038"/>
+  <limit lower="-0.5236" upper="0.5236" effort="100" velocity="1.0"/>
+</joint>
+<joint name="��] 285" type="revolute">
+  <origin xyz="-0.013397 -0.012011 -0.004041" rpy="0 0 0"/>
+  <parent link="L_ankle_xl_2"/>
+  <child link="L_ankle_2"/>
+  <axis xyz="-0.071895 0.997404 -0.004038"/>
+  <limit lower="-0.5236" upper="0.5236" effort="100" velocity="1.0"/>
+</joint>
+<joint name="��] 244" type="revolute">
+  <origin xyz="-0.036704 0.154195 -0.016398" rpy="0 0 0"/>
+  <parent link="ankle_link_2_2"/>
+  <child link="R_bionic_biped_robot_ankle_bar_1"/>
+  <axis xyz="0.071895 -0.997404 0.004038"/>
+  <limit lower="-0.5236" upper="0.5236" effort="100" velocity="1.0"/>
+</joint>
+<joint name="��] 245" type="revolute">
+  <origin xyz="0.073044 -0.130882 -0.073202" rpy="0 0 0"/>
+  <parent link="R_bionic_biped_robot_ankle_bar_1"/>
+  <child link="R_ankle_bar_parts_1"/>
+  <axis xyz="-0.071895 0.997404 -0.004038"/>
+  <limit lower="-0.5236" upper="0.5236" effort="100" velocity="1.0"/>
+</joint>
+<joint name="��] 288" type="revolute">
+  <origin xyz="-0.02423 -0.018855 -0.015698" rpy="0 0 0"/>
+  <parent link="ankle_link_2_1"/>
+  <child link="L_bionic_biped_robot_ankle_bar_v2_1"/>
+  <axis xyz="-0.071895 0.997404 -0.004038"/>
+  <limit lower="-0.5236" upper="0.5236" effort="100" velocity="1.0"/>
+</joint>
+<joint name="��] 294" type="revolute">
+  <origin xyz="0.062297 0.000176 -0.074829" rpy="0 0 0"/>
+  <parent link="L_bionic_biped_robot_ankle_bar_v2_1"/>
+  <child link="L_ankle_bar_parts_v1_1"/>
+  <axis xyz="-0.071895 0.997404 -0.004038"/>
+  <limit lower="-0.5236" upper="0.5236" effort="100" velocity="1.0"/>
+</joint>
 <joint name="��] 249" type="revolute">
   <origin xyz="0.010519 -0.134088 0.001069" rpy="0 0 0"/>
@@ -1156,10 +1198,4 @@
   <child link="R_ankle_xl_2"/>
 </joint>
-<joint name="��] 241" type="continuous">
-  <origin xyz="-0.005236 -0.125216 -0.003583" rpy="0 0 0"/>
-  <parent link="R_ankle_xl_2"/>
-  <child link="R_ankle_2"/>
-  <axis xyz="0.071895 -0.997404 0.004038"/>
-</joint>
 <joint name="���� 242" type="fixed">
   <origin xyz="-0.000144 0.001995 -8e-06" rpy="0 0 0"/>
@@ -1171,16 +1207,4 @@
   <parent link="R_ankle_2"/>
   <child link="ankle_link_2_2"/>
-</joint>
-<joint name="��] 244" type="continuous">
-  <origin xyz="-0.036704 0.154195 -0.016398" rpy="0 0 0"/>
-  <parent link="ankle_link_2_2"/>
-  <child link="R_bionic_biped_robot_ankle_bar_1"/>
-  <axis xyz="0.071895 -0.997404 0.004038"/>
-</joint>
-<joint name="��] 245" type="continuous">
-  <origin xyz="0.073044 -0.130882 -0.073202" rpy="0 0 0"/>
-  <parent link="R_bionic_biped_robot_ankle_bar_1"/>
-  <child link="R_ankle_bar_parts_1"/>
-  <axis xyz="-0.071895 0.997404 -0.004038"/>
 </joint>
 <joint name="���� 246" type="fixed">
@@ -1276,10 +1300,4 @@
   <child link="L_ankle_xl_2"/>
 </joint>
-<joint name="��] 285" type="continuous">
-  <origin xyz="-0.013397 -0.012011 -0.004041" rpy="0 0 0"/>
-  <parent link="L_ankle_xl_2"/>
-  <child link="L_ankle_2"/>
-  <axis xyz="-0.071895 0.997404 -0.004038"/>
-</joint>
 <joint name="���� 286" type="fixed">
   <origin xyz="-0.002588 0.035907 -0.000145" rpy="0 0 0"/>
@@ -1292,10 +1310,4 @@
   <child link="ankle_link_1_1"/>
 </joint>
-<joint name="��] 288" type="continuous">
-  <origin xyz="-0.02423 -0.018855 -0.015698" rpy="0 0 0"/>
-  <parent link="ankle_link_2_1"/>
-  <child link="L_bionic_biped_robot_ankle_bar_v2_1"/>
-  <axis xyz="-0.071895 0.997404 -0.004038"/>
-</joint>
 <joint name="���� 289" type="fixed">
   <origin xyz="0.012586 0.000824 -0.020418" rpy="0 0 0"/>
@@ -1313,10 +1325,4 @@
   <child link="shaft_4"/>
 </joint>
-<joint name="��] 294" type="continuous">
-  <origin xyz="0.062297 0.000176 -0.074829" rpy="0 0 0"/>
-  <parent link="L_bionic_biped_robot_ankle_bar_v2_1"/>
-  <child link="L_ankle_bar_parts_v1_1"/>
-  <axis xyz="-0.071895 0.997404 -0.004038"/>
-</joint>
 <joint name="���� 295" type="fixed">
   <origin xyz="-0.015646 0.005867 -0.00586" rpy="0 0 0"/>
