Commit message: update dql

File: simulation/urdf/mikkelsen2d_description/urdf/mikkelsen2d.xacro (robot description, xacro)
@@ -13,5 +13,5 @@
 <link name="z_prismatic">
   <inertial>
-    <mass value="100"/>
+    <mass value="80"/>
     <inertia ixx="0.2125" ixy="-0.005" ixz="0.0225" iyy="0.205" iyz="0.045" izz="0.0125"/>
     <origin rpy="0 0 0" xyz="0 0 0"/>

Commit message: update dql

File: simulation/urdf/mikkelsen2d_description/urdf/mikkelsen2d.xacro (robot description, xacro)
@@ -13,5 +13,5 @@
 <link name="z_prismatic">
   <inertial>
-    <mass value="80"/>
+    <mass value="75"/>
     <inertia ixx="0.2125" ixy="-0.005" ixz="0.0225" iyy="0.205" iyz="0.045" izz="0.0125"/>
     <origin rpy="0 0 0" xyz="0 0 0"/>
@@ -27,5 +27,5 @@
 <link name="x_prismatic">
   <inertial>
-    <mass value="0.01"/>
+    <mass value="0.001"/>
     <inertia ixx="0.2125" ixy="-0.005" ixz="0.0225" iyy="0.205" iyz="0.045" izz="0.0125"/>
     <origin rpy="0 0 0" xyz="0 0 0"/>
